File: cad/oscillator/oscillator.kicad_sch (KiCad schematic)
At the start: 19 parts, among them P2 Supply-Mode Jumper, U1 LM7805_TO220, U2 74LS00, Y1 DIL-14 VCXO 10Mhz

Commit message: Oscillator Updates
Parts:
- added J1: Molex 22-17-3102, symbol Connector_Generic:Conn_02x10_Top_Bottom
- C1, C2, C3, C4, C5, C6, C7, C8: footprint (none) -> Capacitor_THT:C_Axial_L5.1mm_D3.1mm_P10.00mm_Horizontal
- U1: footprint Package_TO_SOT_THT:TO-220-3_Vertical -> Package_TO_SOT_THT:TO-220-3_Horizontal_TabUp
- U2: footprint (none) -> Package_DIP:CERDIP-14_W7.62mm_SideBrazed
- Y1: footprint Oscillator:Oscillator_SMD_Abracon_ABLNO -> Oscillator:Oscillator_DIP-14; symbol Oscillator:ABLNO -> Oscillator:GTXO-14V
Connections:
- net GND: now also Y1.7 (GND), J1.10 (Pin_10), J1.8 (Pin_8), J1.9 (Pin_9); no longer Y1.2 (GND)
- net at C8.2: now also J1.6 (Pin_6)
- net at C3.1, C4.1, C5.2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: now also Y1.14 (Vcc); no longer Y1.4 (VDD)
- net at U2.2: now also Y1.8 (OUT); no longer Y1.3 (RFout)
- net at P2.1 (A): now also J1.7 (Pin_7)
- net at P2.3 (B), R1.1: now also J1.4 (Pin_4)
Other:
- note added: "Notes: 1) Trimmer R2 and capacitor C6 are for VCXO fine adjust only. If a TCXO is used, remove R2 and replace C6 with wire jumper. 2) For U2, the following can be used: 74LS00, 74F00 (TTL standard), 74HCT00, 74AHCT00 (low consumption CMOS). 3) All resistors a 0.25W. All capacitors are MLCC 50V. D2 is 0.5W. 4) Jumper P2 supply modes: 1-2 = ON/Standby mode (with power switch OFF, TCXO remains activ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"
- moved on the sheet: C1, C2, C3, C4, C5, C6, C7, C8, D1, D2, F1, P2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

Commit message: Oscillator Updates
Parts:
- C1, C2, C3, C4, C5, C6, C7, C8: footprint Capacitor_THT:C_Axial_L5.1mm_D3.1mm_P10.00mm_Horizontal -> Capacitor_THT:C_Axial_L3.8mm_D2.6mm_P10.00mm_Horizontal
- D1, D2: footprint (none) -> Diode_THT:D_A-405_P10.16mm_Horizontal
- F1: footprint (none) -> Fuse:Fuse_Littelfuse_372_D8.50mm
- J1: footprint (none) -> Connector_PinHeader_2.54mm:PinHeader_2x10_P2.54mm_Vertical
- P2: footprint (none) -> Connector_PinSocket_2.54mm:PinSocket_1x03_P2.54mm_Vertical
- R1, R4, R5: footprint (none) -> Resistor_THT:R_Axial_DIN0207_L6.3mm_D2.5mm_P10.16mm_Horizontal
- R2: footprint (none) -> Potentiometer_THT:Potentiometer_Bourns_3296W_Vertical
- U1: footprint Package_TO_SOT_THT:TO-220-3_Horizontal_TabUp -> Package_TO_SOT_THT:TO-220-3_Horizontal_TabDown
Changed lines of the file:
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@@
 			)
 		)
-		(property "Footprint" "Capacitor_THT:C_Axial_L5.1mm_D3.1mm_P10.00mm_Horizontal"
+		(property "Footprint" "Capacitor_THT:C_Axial_L3.8mm_D2.6mm_P10.00mm_Horizontal"
 			(at 200.66 99.3648 0)
 			(effects
@@
 			)
 		)
-		(property "Footprint" "Capacitor_THT:C_Axial_L5.1mm_D3.1mm_P10.00mm_Horizontal"
+		(property "Footprint" "Capacitor_THT:C_Axial_L3.8mm_D2.6mm_P10.00mm_Horizontal"
 			(at 182.5752 54.61 0)
 			(effects
@@
 			)
 		)
-		(property "Footprint" "Capacitor_THT:C_Axial_L5.1mm_D3.1mm_P10.00mm_Horizontal"
+		(property "Footprint" "Capacitor_THT:C_Axial_L3.8mm_D2.6mm_P10.00mm_Horizontal"
 			(at 196.5452 54.61 0)
 			(effects
@@
 			)
 		)
-		(property "Footprint" "Capacitor_THT:C_Axial_L5.1mm_D3.1mm_P10.00mm_Horizontal"
+		(property "Footprint" "Capacitor_THT:C_Axial_L3.8mm_D2.6mm_P10.00mm_Horizontal"
 			(at 148.2852 54.61 0)
 			(effects
@@
 			)
 		)
-		(property "Footprint" "Capacitor_THT:C_Axial_L5.1mm_D3.1mm_P10.00mm_Horizontal"
+		(property "Footprint" "Capacitor_THT:C_Axial_L3.8mm_D2.6mm_P10.00mm_Horizontal"
 			(at 135.5852 54.61 0)
 			(effects
@@
 			)
 		)
-		(property "Footprint" ""
+		(property "Footprint" "Fuse:Fuse_Littelfuse_372_D8.50mm"
 			(at 208.28 48.768 90)
 			(effects
@@
 			)
 		)
-		(property "Footprint" "Capacitor_THT:C_Axial_L5.1mm_D3.1mm_P10.00mm_Horizontal"
+		(property "Footprint" "Capacitor_THT:C_Axial_L3.8mm_D2.6mm_P10.00mm_Horizontal"
 			(at 69.5452 110.49 0)
 			(effects
@@
 			)
 		)
-		(property "Footprint" ""
+		(property "Footprint" "Connector_PinHeader_2.54mm:PinHeader_2x10_P2.54mm_Vertical"
 			(at 241.3 105.41 0)
 			(effects
@@
 			)
 		)
-		(property "Footprint" "Capacitor_THT:C_Axial_L5.1mm_D3.1mm_P10.00mm_Horizontal"
+		(property "Footprint" "Capacitor_THT:C_Axial_L3.8mm_D2.6mm_P10.00mm_Horizontal"
 			(at 155.9052 88.9 0)
 			(effects
@@
 			)
 		)
-		(property "Footprint" ""
+		(property "Footprint" "Resistor_THT:R_Axial_DIN0207_L6.3mm_D2.5mm_P10.16mm_Horizontal"
 			(at 177.292 85.09 90)
 			(effects
@@
 			)
 		)
-		(property "Footprint" "Capacitor_THT:C_Axial_L5.1mm_D3.1mm_P10.00mm_Horizontal"
+		(property "Footprint" "Capacitor_THT:C_Axial_L3.8mm_D2.6mm_P10.00mm_Horizontal"
 			(at 85.09 77.7748 0)
 			(effects
@@
 			)
 		)
-		(property "Footprint" ""
+		(property "Footprint" "Connector_PinSocket_2.54mm:PinSocket_1x03_P2.54mm_Vertical"
 			(at 222.25 66.04 0)
 			(effects
@@
 			)
 		)
-		(property "Footprint" ""
+		(property "Footprint" "Diode_THT:D_A-405_P10.16mm_Horizontal"
 			(at 167.64 85.09 0)
 			(effects
@@
 			)
 		)
-		(property "Footprint" ""
+		(property "Footprint" "Resistor_THT:R_Axial_DIN0207_L6.3mm_D2.5mm_P10.16mm_Horizontal"
 			(at 177.292 71.12 90)
 			(effects
@@
 			)
 		)
-		(property "Footprint" ""
+		(property "Footprint" "Resistor_THT:R_Axial_DIN0207_L6.3mm_D2.5mm_P10.16mm_Horizontal"
 			(at 153.162 105.41 90)
 			(effects
@@
 			)
 		)
-		(property "Footprint" ""
+		(property "Footprint" "Diode_THT:D_A-405_P10.16mm_Horizontal"
 			(at 124.46 50.8 0)
 			(effects
@@
 			)
 		)
-		(property "Footprint" ""
+		(property "Footprint" "Potentiometer_THT:Potentiometer_Bourns_3296W_Vertical"
 			(at 55.88 102.87 0)
 			(effects
@@
 			)
 		)
-		(property "Footprint" "Package_TO_SOT_THT:TO-220-3_Horizontal_TabUp"
+		(property "Footprint" "Package_TO_SOT_THT:TO-220-3_Horizontal_TabDown"
 			(at 167.64 41.275 0)
 			(effects
